File: nanobone.brd (EAGLE design)
At the start: 86.5 x 59.7 mm, 25 parts

Commit message: BOM done.
Parts:
- LED1: value (none) -> blue
- LED2: value (none) -> green
- R6: value 4.75K -> 150
- R8: value 4.75K -> 50
Changed lines of the file:
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@@
 <element name="P9" library="BoneCapeParts" package="FE23-2_SMD" value="" x="43.815" y="5.6134" locked="yes" smashed="yes" rot="MR180">
 <attribute name="OC_NEWARK" value="unknown" x="43.815" y="5.6134" size="1.778" layer="28" rot="MR180" display="off"/>
-<attribute name="MPN" value="" x="43.815" y="5.6134" size="1.778" layer="28" rot="MR180" display="off"/>
+<attribute name="MPN" value="NPPC232KFMS-RC" x="43.815" y="5.6134" size="1.778" layer="28" rot="MR180" display="off"/>
 <attribute name="MF" value="" x="43.815" y="5.6134" size="1.778" layer="28" rot="MR180" display="off"/>
 <attribute name="OC_FARNELL" value="unknown" x="43.815" y="5.6134" size="1.778" layer="28" rot="MR180" display="off"/>
@@
 <element name="P8" library="BoneCapeParts" package="FE23-2_SMD" value="" x="43.815" y="53.8734" locked="yes" smashed="yes" rot="MR180">
 <attribute name="OC_NEWARK" value="unknown" x="43.815" y="53.8734" size="1.778" layer="28" rot="MR180" display="off"/>
-<attribute name="MPN" value="" x="43.815" y="53.8734" size="1.778" layer="28" rot="MR180" display="off"/>
+<attribute name="MPN" value="NPPC232KFMS-RC" x="43.815" y="53.8734" size="1.778" layer="28" rot="MR180" display="off"/>
 <attribute name="MF" value="" x="43.815" y="53.8734" size="1.778" layer="28" rot="MR180" display="off"/>
 <attribute name="OC_FARNELL" value="unknown" x="43.815" y="53.8734" size="1.778" layer="28" rot="MR180" display="off"/>
@@
 <attribute name="NAME" x="71.882" y="27.2034" size="0.635" layer="26" ratio="20" rot="MR90"/>
 <attribute name="VALUE" x="71.628" y="25.2984" size="1.27" layer="28" rot="MR90"/>
+<attribute name="MPN" value="CAT24C256WI-GT3" x="75.565" y="27.2034" size="1.778" layer="28" rot="MR0" display="off"/>
 </element>
 <element name="S1" library="switch-dil" package="CTS-219-02" value="219-02" x="79.7052" y="37.9984" locked="yes" smashed="yes" rot="MR270">
 <attribute name="OC_NEWARK" value="unknown" x="79.7052" y="37.9984" size="1.778" layer="28" rot="MR270" display="off"/>
-<attribute name="MPN" value="" x="79.7052" y="37.9984" size="1.778" layer="28" rot="MR270" display="off"/>
+<attribute name="MPN" value="219-2MST" x="79.7052" y="37.9984" size="1.778" layer="28" rot="MR270" display="off"/>
 <attribute name="MF" value="" x="79.7052" y="37.9984" size="1.778" layer="28" rot="MR270" display="off"/>
 <attribute name="OC_FARNELL" value="unknown" x="79.7052" y="37.9984" size="1.778" layer="28" rot="MR270" display="off"/>
@@
 <element name="C1" library="rcl" package="C0603" value="0.1u" x="80.01" y="44.3484" locked="yes" smashed="yes" rot="MR0">
 <attribute name="NAME" x="80.645" y="44.9834" size="0.635" layer="26" ratio="20" rot="MR0"/>
+<attribute name="MPN" value="VJ0603V104ZXXCW1BC" x="80.01" y="44.3484" size="1.778" layer="28" rot="MR0" display="off"/>
 </element>
 <element name="R3" library="rcl" package="R0603" value="5.6K, 5%" x="76.2" y="32.9184" locked="yes" smashed="yes" rot="MR180">
 <attribute name="NAME" x="75.565" y="32.2834" size="0.635" layer="26" ratio="20" rot="MR180"/>
+<attribute name="MPN" value="RK73B1JTTDD562J" x="76.2" y="32.9184" size="1.778" layer="28" rot="MR180" display="off"/>
 </element>
 <element name="R7" library="rcl" package="R0603" value="4.75K" x="77.47" y="20.2184" locked="yes" smashed="yes" rot="MR270">
 <attribute name="NAME" x="76.835" y="20.8534" size="0.635" layer="26" ratio="20" rot="MR270"/>
+<attribute name="MPN" value="CR0603-FX-4751GLF" x="77.47" y="20.2184" size="1.778" layer="28" rot="MR270" display="off"/>
 </element>
 <element name="R9" library="rcl" package="R0603" value="10K" x="80.01" y="27.8384" locked="yes" smashed="yes" rot="MR270">
 <attribute name="NAME" x="79.375" y="28.4734" size="0.635" layer="26" ratio="20" rot="MR270"/>
+<attribute name="MPN" value="WR06X1002FTL" x="80.01" y="27.8384" size="1.778" layer="28" rot="MR270" display="off"/>
 </element>
 <element name="R1" library="rcl" package="R0603" value="5.6K, 5%" x="77.47" y="16.4084" locked="yes" smashed="yes" rot="MR90">
 <attribute name="NAME" x="78.105" y="15.7734" size="0.635" layer="26" ratio="20" rot="MR90"/>
+<attribute name="MPN" value="RK73B1JTTDD562J" x="77.47" y="16.4084" size="1.778" layer="28" rot="MR90" display="off"/>
 </element>
 <element name="R2" library="rcl" package="R0603" value="4.75K" x="74.93" y="20.2184" locked="yes" smashed="yes" rot="MR270">
 <attribute name="NAME" x="74.295" y="20.8534" size="0.635" layer="26" ratio="20" rot="MR270"/>
+<attribute name="MPN" value="CR0603-FX-4751GLF" x="74.93" y="20.2184" size="1.778" layer="28" rot="MR270" display="off"/>
 </element>
 <element name="R4" library="rcl" package="R0603" value="4.75K, DNI" x="72.39" y="20.2184" locked="yes" smashed="yes" rot="MR270">
 <attribute name="NAME" x="71.755" y="20.8534" size="0.635" layer="26" ratio="20" rot="MR270"/>
+<attribute name="MPN" value="CR0603-FX-4751GLF" x="72.39" y="20.2184" size="1.778" layer="28" rot="MR270" display="off"/>
 </element>
 <element name="R5" library="rcl" package="R0603" value="4.75K" x="74.93" y="16.4084" locked="yes" smashed="yes" rot="MR270">
 <attribute name="NAME" x="74.295" y="17.0434" size="0.635" layer="26" ratio="20" rot="MR270"/>
+<attribute name="MPN" value="CR0603-FX-4751GLF" x="74.93" y="16.4084" size="1.778" layer="28" rot="MR270" display="off"/>
 </element>
 <element name="SV1" library="BoneCapeParts" package="FE20-2" value="" x="48.895" y="51.3334" locked="yes" smashed="yes" rot="R180">
 <attribute name="OC_NEWARK" value="unknown" x="48.895" y="51.3334" size="1.778" layer="27" rot="R180" display="off"/>
-<attribute name="MPN" value="" x="48.895" y="51.3334" size="1.778" layer="27" rot="R180" display="off"/>
+<attribute name="MPN" value="NPPC202KFMS-RC" x="48.895" y="51.3334" size="1.778" layer="27" rot="R180" display="off"/>
 <attribute name="MF" value="" x="48.895" y="51.3334" size="1.778" layer="27" rot="R180" display="off"/>
 <attribute name="OC_FARNELL" value="unknown" x="48.895" y="51.3334" size="1.778" layer="27" rot="R180" display="off"/>
@@
 <element name="SV2" library="BoneCapeParts" package="FE20-2" value="" x="48.895" y="8.1534" locked="yes" smashed="yes">
 <attribute name="OC_NEWARK" value="unknown" x="48.895" y="8.1534" size="1.778" layer="27" display="off"/>
-<attribute name="MPN" value="" x="48.895" y="8.1534" size="1.778" layer="27" display="off"/>
+<attribute name="MPN" value="NPPC202KFMS-RC" x="48.895" y="8.1534" size="1.778" layer="27" display="off"/>
 <attribute name="MF" value="" x="48.895" y="8.1534" size="1.778" layer="27" display="off"/>
 <attribute name="OC_FARNELL" value="unknown" x="48.895" y="8.1534" size="1.778" layer="27" display="off"/>
@@
 <attribute name="VALUE" x="0.57710625" y="4.17655625" size="1.27" layer="27" font="vector" rot="R315"/>
 </element>
-<element name="LED1" library="led" package="CHIPLED_0603" value="" x="81.28" y="35.4584" locked="yes" smashed="yes" rot="R180">
+<element name="LED1" library="led" package="CHIPLED_0603" value="blue" x="81.28" y="35.4584" locked="yes" smashed="yes" rot="R180">
 <attribute name="NAME" x="81.915" y="36.7284" size="0.635" layer="25" ratio="20" rot="R270"/>
 <attribute name="VALUE" x="79.375" y="36.7284" size="1.27" layer="27" rot="R270"/>
+<attribute name="MPN" value="HT-193NB-5589" x="81.28" y="35.4584" size="1.778" layer="27" rot="R180" display="off"/>
 </element>
-<element name="R6" library="rcl" package="R0603" value="4.75K" x="82.55" y="32.9184" locked="yes" smashed="yes" rot="MR0">
+<element name="R6" library="rcl" package="R0603" value="150" x="82.55" y="32.9184" locked="yes" smashed="yes" rot="MR0">
 <attribute name="NAME" x="83.185" y="33.5534" size="0.635" layer="26" ratio="20" rot="MR0"/>
+<attribute name="MPN" value="302-150-RC" x="82.55" y="32.9184" size="1.778" layer="28" rot="MR0" display="off"/>
 </element>
-<element name="LED2" library="led" package="CHIPLED_0603" value="" x="81.28" y="22.7584" locked="yes" smashed="yes">
+<element name="LED2" library="led" package="CHIPLED_0603" value="green" x="81.28" y="22.7584" locked="yes" smashed="yes">
 <attribute name="NAME" x="82.55" y="22.1234" size="0.635" layer="25" ratio="20" rot="R90"/>
 <attribute name="VALUE" x="83.185" y="21.4884" size="1.27" layer="27" rot="R90"/>
+<attribute name="MPN" value="LG Q971-KN-1" x="81.28" y="22.7584" size="1.778" layer="27" display="off"/>
 </element>
-<element name="R8" library="rcl" package="R0603" value="4.75K" x="81.28" y="22.7584" locked="yes" smashed="yes" rot="MR90">
+<element name="R8" library="rcl" package="R0603" value="50" x="81.28" y="22.7584" locked="yes" smashed="yes" rot="MR90">
 <attribute name="NAME" x="81.915" y="22.1234" size="0.635" layer="26" ratio="20" rot="MR90"/>
+<attribute name="MPN" value="302-49.9-RC" x="81.28" y="22.7584" size="1.778" layer="28" rot="MR90" display="off"/>
 </element>
 <element name="SV3" library="con-lstb" package="MA03-1" value="" x="2.54" y="13.2334" locked="yes" smashed="yes" rot="R90">
