File: nanobone.sch (EAGLE design)
At the start: 25 parts

Commit message: BOM done.
Parts:
- C1: MPN (none) -> VJ0603V104ZXXCW1BC
- LED1: value (none) -> blue; MPN (none) -> HT-193NB-5589
- LED2: value (none) -> green; MPN (none) -> LG Q971-KN-1
- P8, P9: MPN (none) -> NPPC232KFMS-RC
- R1, R3: MPN (none) -> RK73B1JTTDD562J
- R2, R4, R5, R7: MPN (none) -> CR0603-FX-4751GLF
- R6: value 4.75K -> 150; MPN (none) -> 302-150-RC
- R8: value 4.75K -> 50; MPN (none) -> 302-49.9-RC
- R9: MPN (none) -> WR06X1002FTL
- S1: MPN (none) -> 219-2MST
- SV1, SV2: MPN (none) -> NPPC202KFMS-RC
- U$1: MPN (none) -> CAT24C256WI-GT3
Other:
- note added: "NanoBone"
- note removed: "Cape Name"
- moved on the sheet: LED1, LED2, R6, R8
